File: POSCON.PCB.brd (EAGLE design)
At the start: 55.8 x 40.9 mm, 27 parts, among them J1-PROG RJ45-8, J2 RJ45-8, U1 MC9S08QG-DT, U3 RS485SOIC, U4 PCA9552

Commit message: POSCON.PCB.v1.0
Release version. Moved Gerbers to top level (no production files here!).
Added version name to bottom silk
Other:
- board text added: "POSCON.PCB.v1.0"
Changed lines of the file:
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@@
 <hole x="16.5" y="18" drill="3.9"/>
 <hole x="16.5" y="-18" drill="3.9"/>
+<text x="7.95" y="-18.35" size="1.27" layer="22" rot="MR0">POSCON.PCB.v1.0</text>
 </plain>
 <attributes>
@@
 <attribute name="NOTES" value="DNP" x="21" y="0" size="1.778" layer="27" display="off"/>
 </element>
-<element name="U$1" library="adafruit" package="FIDUCIAL_1MM" value="FIDUCIAL" x="-11.65" y="-18.2"/>
-<element name="U$2" library="adafruit" package="FIDUCIAL_1MM" value="FIDUCIAL" x="11.95" y="-18.4"/>
-<element name="U$6" library="adafruit" package="FIDUCIAL_1MM" value="FIDUCIAL" x="-11.35" y="18.2"/>
-<element name="U$7" library="adafruit" package="FIDUCIAL_1MM" value="FIDUCIAL" x="-11.65" y="-18.2" rot="MR0"/>
-<element name="U$8" library="adafruit" package="FIDUCIAL_1MM" value="FIDUCIAL" x="11.95" y="-18.4" rot="MR0"/>
-<element name="U$9" library="adafruit" package="FIDUCIAL_1MM" value="FIDUCIAL" x="-11.35" y="18.2" rot="MR0"/>
+<element name="U$1" library="adafruit" package="FIDUCIAL_1MM" value="FIDUCIAL" x="-11.65" y="-18.2">
+<attribute name="NOTES" value="DNP" x="-11.65" y="-18.2" size="1.778" layer="27" display="off"/>
+</element>
+<element name="U$2" library="adafruit" package="FIDUCIAL_1MM" value="FIDUCIAL" x="11.95" y="-18.4">
+<attribute name="NOTES" value="DNP" x="11.95" y="-18.4" size="1.778" layer="27" display="off"/>
+</element>
+<element name="U$6" library="adafruit" package="FIDUCIAL_1MM" value="FIDUCIAL" x="-11.35" y="18.2">
+<attribute name="NOTES" value="DNP" x="-11.35" y="18.2" size="1.778" layer="27" display="off"/>
+</element>
+<element name="U$7" library="adafruit" package="FIDUCIAL_1MM" value="FIDUCIAL" x="-11.65" y="-18.2" rot="MR0">
+<attribute name="NOTES" value="DNP" x="-11.65" y="-18.2" size="1.778" layer="28" rot="MR0" display="off"/>
+</element>
+<element name="U$8" library="adafruit" package="FIDUCIAL_1MM" value="FIDUCIAL" x="11.95" y="-18.4" rot="MR0">
+<attribute name="NOTES" value="DNP" x="11.95" y="-18.4" size="1.778" layer="28" rot="MR0" display="off"/>
+</element>
+<element name="U$9" library="adafruit" package="FIDUCIAL_1MM" value="FIDUCIAL" x="-11.35" y="18.2" rot="MR0">
+<attribute name="NOTES" value="DNP" x="-11.35" y="18.2" size="1.778" layer="28" rot="MR0" display="off"/>
+</element>
 </elements>
 <signals>
