File: POSCON.PCB Design Files/POSCON.PCB.brd (EAGLE design)
At the start: 55.8 x 40.9 mm, 27 parts, among them J1-PROG RJ45-8, J2 RJ45-8, U1 MC9S08QG-DT, U3 RS485SOIC, U4 PCA9552

Commit message: Fixing power traces in progress
Not done. Moved components
Parts:
- moved U$1 16.4 mm to (-25.9, -10.1)
- moved U$7 16.4 mm to (-25.9, -10.1)
- moved R.D2C 0.86 mm to (-16.1, -11.2)
Routing:
- net +3V3: track 194.2 -> 253.5 mm, vias 8 -> 13
- net GND: track 84.2 -> 106.3 mm
- net N$35: track 40.8 -> 38.0 mm
- net N$36: track 40.4 -> 37.6 mm
- net N$39: track 4.55 -> 7.26 mm
- net N$40: track 12.8 -> 11.8 mm
- net N$38: track 26.4 -> 25.4 mm
- net N$41: track 6.19 -> 5.43 mm

Commit message: Finished power trace
Changed label to v1.1, fixed traces and moved vias / traces to
accomodate
Parts:
- moved R.D2C 1.23 mm to (-16.6, -10.0)
- moved U$1 0.43 mm to (-26.1, -10.4)
- moved U$7 0.43 mm to (-26.1, -10.4)
Routing:
- net +3V3: track 253.5 -> 278.7 mm
- net GND: track 106.3 -> 90.0 mm, vias 11 -> 16
- net N$40: track 11.8 -> 7.73 mm
- net N$41: track 5.43 -> 8.93 mm
- net N$38: track 25.4 -> 27.6 mm
- net N$39: track 7.26 -> 9.22 mm
- net N$30: track 5.79 -> 7.61 mm
- net N$36: track 37.6 -> 39.1 mm
- net N$37: track 29.6 -> 30.6 mm
- net N$35: track 38.0 -> 38.7 mm
Other:
- board text added: "POSCON.PCB.v1.1"
- board text added: "R.S. 12/30/14"
- board text removed: "POSCON.PCB.v1.0"

Commit message: Prepare for release 1.2
Labelling, part names and numbers, new Gerbers and production documents
Parts:
- U1: value MC9S08QG-DT -> MC9S08SH8CTG
Other:
- board text added: "POSCON.PCB.v1.2"
- board text added: "R.S. 1/6/15"
- board text removed: "POSCON.PCB.v1.1"
- board text removed: "R.S. 12/30/14"
Changed lines of the file:
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@@
 <hole x="16.5" y="18" drill="3.9"/>
 <hole x="16.5" y="-18" drill="3.9"/>
-<text x="7.95" y="-18.05" size="1.27" layer="22" rot="MR0">POSCON.PCB.v1.1</text>
-<text x="7.95" y="-19.7" size="1.27" layer="22" rot="MR0">R.S. 12/30/14</text>
+<text x="7.95" y="-18.05" size="1.27" layer="22" rot="MR0">POSCON.PCB.v1.2</text>
+<text x="7.95" y="-19.7" size="1.27" layer="22" rot="MR0">R.S. 1/6/15</text>
 </plain>
 <attributes>
@@
 <param name="mlMinCreamFrame" value="0mil"/>
 <param name="mlMaxCreamFrame" value="0mil"/>
-<param name="mlViaStopLimit" value="0mil"/>
+<param name="mlViaStopLimit" value="0.5mm"/>
 <param name="srRoundness" value="0"/>
 <param name="srMinRoundness" value="0mil"/>
@@
 </autorouter>
 <elements>
-<element name="U1" library="GW-devices" package="TSSOP16" value="MC9S08QG-DT" x="16.39" y="11.47" smashed="yes" rot="MR90">
+<element name="U1" library="GW-devices" package="TSSOP16" value="MC9S08SH8CTG" x="16.39" y="11.47" smashed="yes" rot="MR90">
 <attribute name="NAME" x="14.9072" y="15.5244" size="1.27" layer="22" ratio="10" rot="MR180"/>
 <attribute name="MFGN" value="Freescale" x="16.39" y="11.47" size="1.778" layer="28" rot="MR90" display="off"/>
-<attribute name="MFGP" value="MC9S08QG8CDTER" x="16.39" y="11.47" size="1.778" layer="28" rot="MR90" display="off"/>
-<attribute name="PRICE" value="1.73" x="16.39" y="11.47" size="1.778" layer="28" rot="MR90" display="off"/>
+<attribute name="MFGP" value="MC9S08SH8CTG" x="16.39" y="11.47" size="1.778" layer="28" rot="MR90" display="off"/>
+<attribute name="PRICE" value="2.00" x="16.39" y="11.47" size="1.778" layer="28" rot="MR90" display="off"/>
 </element>
 <element name="C1" library="GW-devices" package="C0402" value=".1uF" x="9.98" y="12.56" smashed="yes" rot="MR270">
@@
 <element name="R.D2D" library="GW-devices" package="3216-4X" value="RESISTOR-ARRAY-4X-3216" x="-5.9" y="-12.7" smashed="yes" rot="MR0">
 <attribute name="MFGN" value="Yageo" x="-0.4" y="8.8" size="1.778" layer="28" rot="MR0" display="off"/>
-<attribute name="MFGP" value="YC164-JR-07120RL" x="-0.4" y="8.8" size="1.778" layer="28" rot="MR0" display="off"/>
+<attribute name="MFGP" value="YC164-JR-07620RL" x="-0.4" y="8.8" size="1.778" layer="28" rot="MR0" display="off"/>
 <attribute name="PRICE" value="0.006" x="-0.4" y="8.8" size="1.778" layer="28" rot="MR0" display="off"/>
 <attribute name="NAME" x="-4" y="-10.95" size="1.27" layer="22" ratio="10" rot="MR0"/>
@@
 <element name="R.D2C" library="GW-devices" package="3216-4X" value="RESISTOR-ARRAY-4X-3216" x="-16.6" y="-10" smashed="yes" rot="MR0">
 <attribute name="MFGN" value="Yageo" x="-16.6" y="7" size="1.778" layer="28" rot="MR0" display="off"/>
-<attribute name="MFGP" value="YC164-JR-07120RL" x="-16.6" y="7" size="1.778" layer="28" rot="MR0" display="off"/>
+<attribute name="MFGP" value="YC164-JR-07620RL" x="-16.6" y="7" size="1.778" layer="28" rot="MR0" display="off"/>
 <attribute name="PRICE" value="0.006" x="-16.6" y="7" size="1.778" layer="28" rot="MR0" display="off"/>
 <attribute name="NAME" x="-14.8" y="-13.05" size="1.27" layer="22" ratio="10" rot="MR0"/>
@@
 <element name="R.D2A" library="GW-devices" package="3216-4X" value="RESISTOR-ARRAY-4X-3216" x="-5.6" y="13" smashed="yes" rot="MR0">
 <attribute name="MFGN" value="Yageo" x="5.9" y="17" size="1.778" layer="28" rot="MR0" display="off"/>
-<attribute name="MFGP" value="YC164-JR-07120RL" x="5.9" y="17" size="1.778" layer="28" rot="MR0" display="off"/>
+<attribute name="MFGP" value="YC164-JR-07620RL" x="5.9" y="17" size="1.778" layer="28" rot="MR0" display="off"/>
 <attribute name="PRICE" value="0.006" x="5.9" y="17" size="1.778" layer="28" rot="MR0" display="off"/>
 <attribute name="NAME" x="-3.45" y="14.75" size="1.27" layer="22" ratio="10" rot="MR0"/>
@@
 <element name="R.D2B" library="GW-devices" package="3216-4X" value="RESISTOR-ARRAY-4X-3216" x="-16" y="12.4" smashed="yes" rot="MR0">
 <attribute name="MFGN" value="Yageo" x="1" y="11.9" size="1.778" layer="28" rot="MR0" display="off"/>
-<attribute name="MFGP" value="YC164-JR-07120RL" x="1" y="11.9" size="1.778" layer="28" rot="MR0" display="off"/>
+<attribute name="MFGP" value="YC164-JR-07620RL" x="1" y="11.9" size="1.778" layer="28" rot="MR0" display="off"/>
 <attribute name="PRICE" value="0.006" x="1" y="11.9" size="1.778" layer="28" rot="MR0" display="off"/>
 <attribute name="NAME" x="-13.55" y="14.05" size="1.27" layer="22" ratio="10" rot="MR0"/>
@@
 <wire x1="-7.2" y1="-17.15" x2="-8.5" y2="-17.15" width="2" layer="1"/>
 <wire x1="-8.5" y1="-17.15" x2="-9.85" y2="-17.15" width="2" layer="1"/>
-<via x="-8.5" y="-17.15" extent="1-16" drill="0.6"/>
-<via x="-9.85" y="-17.15" extent="1-16" drill="0.6"/>
-<via x="-11.15" y="-17.15" extent="1-16" drill="0.6"/>
+<via x="-8.5" y="-17.15" extent="1-16" drill="0.5"/>
+<via x="-9.85" y="-17.15" extent="1-16" drill="0.5"/>
+<via x="-11.15" y="-17.15" extent="1-16" drill="0.5"/>
 <wire x1="-11.45" y1="-17.15" x2="-13.275" y2="-15.325" width="2" layer="16"/>
 <wire x1="-13.275" y1="-15.325" x2="-13.35" y2="-15.25" width="1.5" layer="16"/>
@@
 <wire x1="19.2" y1="3.9" x2="18.7" y2="4.4" width="1" layer="16"/>
 <wire x1="17.9" y1="4.45" x2="18.65" y2="4.45" width="1" layer="16"/>
-<wire x1="18.65" y1="4.45" x2="18.7" y2="4.4" width="0.8128" layer="16"/>
+<wire x1="18.65" y1="4.45" x2="18.7" y2="4.4" width="1" layer="16"/>
 <wire x1="18.7" y1="-5.75" x2="18.7" y2="-5.7" width="2" layer="1"/>
 <wire x1="19.2" y1="-4.6" x2="19.2" y2="-4.5" width="2" layer="1"/>
@@
 </signal>
 </signals>
+<errors>
+</errors>
 </board>
 </drawing>

Commit message: Fixing DRC
Residual Eagle errors on checklist
Parts:
- moved R5 0.16 mm to (4.04, 9.22)
Connections:
- net N$19 renamed DIR
- net N$23 renamed RST
- net N$3 renamed LED_DI
- net N$42 renamed ACK
- net N$43 renamed INC_UP
- net N$45 renamed INC_DOWN
- net N$9 renamed BDM
- net SLA renamed SDA
- net SLC renamed SCL
Changed lines of the file:
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@@
 <setting verticaltext="up"/>
 </settings>
-<grid distance="0.05" unitdist="mm" unit="mm" style="lines" multiple="1" display="yes" altdistance="0.003125" altunitdist="mic" altunit="mm"/>
+<grid distance="0.00196850394" unitdist="inch" unit="inch" style="lines" multiple="1" display="yes" altdistance="0.000000123031" altunitdist="inch" altunit="inch"/>
 <layers>
 <layer number="1" name="Top" color="4" fill="1" visible="yes" active="yes"/>
@@
 <attribute name="NAME" x="-13.55" y="14.05" size="1.27" layer="22" ratio="10" rot="MR0"/>
 </element>
-<element name="R5" library="GW-devices" package="RF-R0402" value="10K" x="4" y="9.37" smashed="yes" rot="MR90">
-<attribute name="MFGN" value="Panasonic" x="7" y="-1.13" size="1.778" layer="28" rot="MR90" display="off"/>
-<attribute name="MFGP" value="ERJ-2GEJ103X" x="7" y="-1.13" size="1.778" layer="28" rot="MR90" display="off"/>
-<attribute name="PRICE" value="0.02" x="7" y="-1.13" size="1.778" layer="28" rot="MR90" display="off"/>
-<attribute name="NAME" x="5.03" y="10.2" size="1.27" layer="22" ratio="10" rot="MR0"/>
-<attribute name="VALUE" x="2.25" y="8.37" size="1.27" layer="28" rot="MR90"/>
+<element name="R5" library="GW-devices" package="RF-R0402" value="10K" x="4.037684375" y="9.219246875" smashed="yes" rot="MR90">
+<attribute name="MFGN" value="Panasonic" x="7.037684375" y="-1.280753125" size="1.778" layer="28" rot="MR90" display="off"/>
+<attribute name="MFGP" value="ERJ-2GEJ103X" x="7.037684375" y="-1.280753125" size="1.778" layer="28" rot="MR90" display="off"/>
+<attribute name="PRICE" value="0.02" x="7.037684375" y="-1.280753125" size="1.778" layer="28" rot="MR90" display="off"/>
+<attribute name="NAME" x="4.979253125" y="10.088759375" size="1.27" layer="22" ratio="10" rot="MR0"/>
 </element>
 <element name="R6" library="GW-devices" package="RF-R0402" value="10K" x="5.25" y="7.92" smashed="yes" rot="MR90">
@@
 <attribute name="PRICE" value="0.02" x="3.75" y="-7.08" size="1.778" layer="28" rot="MR90" display="off"/>
 <attribute name="NAME" x="3.45" y="5.47" size="1.27" layer="22" ratio="10" rot="MR90"/>
-<attribute name="VALUE" x="3.5" y="6.92" size="1.27" layer="28" rot="MR90"/>
-</element>
-<element name="LED2" library="GW-devices" package="7SEGMENT-1DIG-.40-SMD" value="7SEGMENT-1DIGITSMD" x="-5.95" y="0">
+</element>
+<element name="LED2" library="GW-devices" package="7SEGMENT-1DIG-.40-SMD" value="7SEGMENT-1DIGITSMD" x="-5.95" y="0" smashed="yes">
 <attribute name="MFGN" value="Kingbright" x="-5.95" y="0" size="1.778" layer="27" display="off"/>
 <attribute name="MFGP" value="ACSA04-41SEKWA-F01 " x="-5.95" y="0" size="1.778" layer="27" display="off"/>
-</element>
-<element name="LED1" library="GW-devices" package="7SEGMENT-1DIG-.40-SMD" value="7SEGMENT-1DIGITSMD" x="-16.15" y="0">
+<attribute name="NAME" x="-0.96" y="-9.01" size="1.27" layer="25"/>
+</element>
+<element name="LED1" library="GW-devices" package="7SEGMENT-1DIG-.40-SMD" value="7SEGMENT-1DIGITSMD" x="-16.15" y="0" smashed="yes">
 <attribute name="MFGN" value="Kingbright" x="-16.15" y="0" size="1.778" layer="27" display="off"/>
 <attribute name="MFGP" value="ACSA04-41SEKWA-F01 " x="-16.15" y="0" size="1.778" layer="27" display="off"/>
+<attribute name="NAME" x="-21.64" y="-3.11" size="1.27" layer="25" rot="R90"/>
 </element>
 <element name="SW-ACK" library="GW-devices" package="SWITCH-TACTILE-320.01E11WHT" value="SWITCH-TACTILE-320.01E11WHT" x="5.45" y="0">
@@
 <attribute name="MFGP" value="320.01E11WHT" x="-7.55" y="15" size="1.778" layer="27" display="off"/>
 </element>
-<element name="U$3" library="GW-devices" package="ESWITCH-TL3301PF" value="SWITCH-TACTILE" x="-13.5" y="-12.75">
+<element name="U$3" library="GW-devices" package="ESWITCH-TL3301PF" value="SWITCH-TACTILE" x="-13.5" y="-12.75" smashed="yes">
 <attribute name="MFGN" value="E-Switch" x="-13.5" y="-12.75" size="1.778" layer="27" display="off"/>
 <attribute name="MFGP" value="TL3301PF160QG" x="-13.5" y="-12.75" size="1.778" layer="27" display="off"/>
-</element>
-<element name="U$4" library="GW-devices" package="ESWITCH-TL3301PF" value="SWITCH-TACTILE" x="-13.5" y="12.75">
+<attribute name="NAME" x="-21.1" y="-13.4" size="1.6764" layer="25"/>
+</element>
+<element name="U$4" library="GW-devices" package="ESWITCH-TL3301PF" value="SWITCH-TACTILE" x="-13.5" y="12.75" smashed="yes">
 <attribute name="MFGN" value="E-Switch" x="-13.5" y="12.75" size="1.778" layer="27" display="off"/>
 <attribute name="MFGP" value="TL3301PF160QG" x="-13.5" y="12.75" size="1.778" layer="27" display="off"/>
+<attribute name="NAME" x="-21.1" y="11.85" size="1.6764" layer="25"/>
 </element>
 <element name="J1-PROG" library="GW-devices" package="MOLEX-0955016649" value="RJ45-8" x="24.435" y="0" smashed="yes" rot="MR270">
@@
 <wire x1="13.4" y1="-4.45" x2="14.205" y2="-4.45" width="1" layer="16"/>
 <wire x1="14.205" y1="-4.45" x2="14.21" y2="-4.445" width="0.254" layer="16"/>
-<wire x1="4" y1="9.87" x2="2.98" y2="9.87" width="0.254" layer="16"/>
 <wire x1="2.98" y1="9.87" x2="2.4" y2="10.45" width="0.254" layer="16"/>
-<wire x1="4" y1="9.87" x2="4.43" y2="9.87" width="0.254" layer="16"/>
-<wire x1="4.43" y1="9.87" x2="5.25" y2="9.05" width="0.254" layer="16"/>
 <wire x1="5.25" y1="9.05" x2="5.25" y2="8.42" width="0.254" layer="16"/>
 <wire x1="-16.15" y1="7.5" x2="-16.15" y2="5.8" width="0.4064" layer="1"/>
@@
 <wire x1="-21.85" y1="2.45" x2="-21.85" y2="1.95" width="1" layer="16"/>
 <wire x1="-21.85" y1="1.95" x2="-19.7" y2="1.95" width="1" layer="16"/>
+<wire x1="2.98" y1="9.87" x2="3.88693125" y2="9.87" width="0.254" layer="16"/>
+<wire x1="3.88693125" y1="9.87" x2="4.037684375" y2="9.719246875" width="0.254" layer="16"/>
+<wire x1="5.25" y1="9.05" x2="5.25" y2="9.1" width="0.254" layer="16"/>
+<wire x1="5.25" y1="9.1" x2="4.55" y2="9.8" width="0.254" layer="16"/>
+<wire x1="4.55" y1="9.8" x2="4.1184375" y2="9.8" width="0.254" layer="16"/>
+<wire x1="4.1184375" y1="9.8" x2="4.037684375" y2="9.719246875" width="0.254" layer="16"/>
 </signal>
 <signal name="TX">
@@
 <wire x1="20.65" y1="-5.75" x2="19.3" y2="-7.1" width="0.254" layer="16"/>
 </signal>
-<signal name="N$19">
+<signal name="DIR">
 <contactref element="U1" pad="9"/>
 <contactref element="U3" pad="2"/>
@@
 <wire x1="-0.002665625" y1="-6.052665625" x2="0.047334375" y2="-6.102665625" width="0.254" layer="1"/>
 </signal>
-<signal name="N$9">
+<signal name="BDM">
 <contactref element="BDM" pad="P$1"/>
 <contactref element="U1" pad="2"/>
@@
 <wire x1="12.35" y1="6.6" x2="12.55" y2="6.8" width="0.254" layer="16"/>
 </signal>
-<signal name="N$23">
+<signal name="RST">
 <contactref element="BDM" pad="P$4"/>
 <contactref element="U1" pad="1"/>
@@
 <wire x1="0.452665625" y1="-5.897334375" x2="0.502665625" y2="-5.947334375" width="0.254" layer="1"/>
 </signal>
-<signal name="SLC">
+<signal name="SCL">
 <contactref element="U4" pad="22"/>
 <contactref element="R6" pad="1"/>
@@
 <wire x1="5" y1="8.5" x2="5.7" y2="8.5" width="0.254" layer="1"/>
 </signal>
-<signal name="SLA">
+<signal name="SDA">
 <contactref element="U4" pad="23"/>
 <contactref element="R5" pad="1"/>
@@
 <wire x1="12.745" y1="12.445" x2="11.5" y2="11.2" width="0.254" layer="16"/>
 <wire x1="11.5" y1="11.2" x2="10.95" y2="11.2" width="0.254" layer="16"/>
-<wire x1="4" y1="8.87" x2="3.02" y2="8.87" width="0.254" layer="16"/>
-<wire x1="3.02" y1="8.87" x2="2.9" y2="8.75" width="0.254" layer="16"/>
 <wire x1="4.1" y1="8.75" x2="2.9" y2="8.75" width="0.254" layer="1"/>
+<wire x1="2.9" y1="8.75" x2="4.00693125" y2="8.75" width="0.254" layer="16"/>
+<wire x1="4.00693125" y1="8.75" x2="4.037684375" y2="8.719246875" width="0.254" layer="16"/>
 </signal>
 <signal name="RESET">
@@
 <wire x1="-19.9" y1="-6.1" x2="-19.9" y2="-4.3" width="0.254" layer="1"/>
 </signal>
-<signal name="N$42">
+<signal name="ACK">
 <contactref element="SW-ACK" pad="P$1"/>
 <contactref element="SW-ACK" pad="P$2"/>
@@
 <wire x1="20.825" y1="10.325" x2="20.825" y2="9.075" width="0.254" layer="16"/>
 </signal>
-<signal name="N$43">
+<signal name="INC_UP">
 <contactref element="U1" pad="15"/>
 <contactref element="U$4" pad="1"/>
@@
 <wire x1="2.42" y1="16.93" x2="2.05" y2="17.3" width="0.254" layer="16"/>
 </signal>
-<signal name="N$45">
+<signal name="INC_DOWN">
 <contactref element="U1" pad="16"/>
 <contactref element="U$3" pad="1"/>
@@
 <wire x1="-11.8" y1="-11.15" x2="-11.8" y2="-11.7" width="0.254" layer="1"/>
 </signal>
-<signal name="N$3">
+<signal name="LED_DI">
 <contactref element="U$5" pad="2"/>
 <contactref element="U1" pad="8"/>

Commit message: New files for release 1.2
For review and sent to quote at AC.
Routing:
- net N$36: track 39.1 -> 40.7 mm
- net N$35: track 38.7 -> 40.3 mm
- net +3V3: track 278.8 -> 279.0 mm, vias 13 -> 15
- net GND: vias 16 -> 19

Commit message: Release v1.3
Fixed silkscreen (pin 1 markers), added WS2812S, added date / name to
fab text and updated all files correspondingly (BOM, ECO)
Parts:
- J1-PROG, J2: device GW-devices:MOLEX-0955016649 -> GW-devices:RJ45_SMD
Connections:
- net +3V3 renamed +5V
Other:
- board text added: "POSCON.PCB.v1.3"
- board text added: "R.S. 3/12/15"
- board text removed: "POSCON.PCB.v1.2"
- board text removed: "R.S. 1/6/15"
Changed lines of the file:
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@@
 <hole x="16.5" y="18" drill="3.9"/>
 <hole x="16.5" y="-18" drill="3.9"/>
-<text x="7.95" y="-18.05" size="1.27" layer="22" rot="MR0">POSCON.PCB.v1.2</text>
-<text x="7.95" y="-19.7" size="1.27" layer="22" rot="MR0">R.S. 1/6/15</text>
+<text x="7.95" y="-18.05" size="1.27" layer="22" rot="MR0">POSCON.PCB.v1.3</text>
+<text x="7.95" y="-19.7" size="1.27" layer="22" rot="MR0">R.S. 3/12/15</text>
 </plain>
 <attributes>
@@
 <attribute name="MFGN" value="E-Switch" x="-13.5" y="-12.75" size="1.778" layer="27" display="off"/>
 <attribute name="MFGP" value="TL3301PF160QG" x="-13.5" y="-12.75" size="1.778" layer="27" display="off"/>
-<attribute name="NAME" x="-21.1" y="-13.4" size="1.6764" layer="25"/>
+<attribute name="NAME" x="-21.35" y="-13.95" size="1.6764" layer="25"/>
 </element>
 <element name="U$4" library="GW-devices" package="ESWITCH-TL3301PF" value="SWITCH-TACTILE" x="-13.5" y="12.75" smashed="yes">
 <attribute name="MFGN" value="E-Switch" x="-13.5" y="12.75" size="1.778" layer="27" display="off"/>
 <attribute name="MFGP" value="TL3301PF160QG" x="-13.5" y="12.75" size="1.778" layer="27" display="off"/>
-<attribute name="NAME" x="-21.1" y="11.85" size="1.6764" layer="25"/>
-</element>
-<element name="J1-PROG" library="GW-devices" package="MOLEX-0955016649" value="RJ45-8" x="24.435" y="0" smashed="yes" rot="MR270">
+<attribute name="NAME" x="-21.6" y="11.5" size="1.6764" layer="25"/>
+</element>
+<element name="J1-PROG" library="GW-devices" package="RJ45_SMD" value="RJ45-8" x="24.435" y="0" smashed="yes" rot="MR270">
 <attribute name="MFGN" value="Molex" x="24.435" y="0" size="1.778" layer="28" rot="MR270" display="off"/>
 <attribute name="MFGP" value="0955016889" x="24.435" y="0" size="1.778" layer="28" rot="MR270" display="off"/>
@@
 <attribute name="NAME" x="16.9672" y="-8.1456" size="1.27" layer="22" ratio="10" rot="MR180"/>
 </element>
-<element name="J2" library="GW-devices" package="MOLEX-0955016649" value="RJ45-8" x="-24.435" y="0" smashed="yes" rot="MR90">
+<element name="J2" library="GW-devices" package="RJ45_SMD" value="RJ45-8" x="-24.435" y="0" smashed="yes" rot="MR90">
 <attribute name="MFGN" value="Molex" x="-24.435" y="0" size="1.778" layer="28" rot="MR90" display="off"/>
 <attribute name="MFGP" value="0955016889" x="-24.435" y="0" size="1.778" layer="28" rot="MR90" display="off"/>
@@
 <element name="U$5" library="GW-devices" package="PLCC-6" value="WS2812" x="21" y="0">
 <attribute name="MFGN" value="Worldsemi" x="21" y="0" size="1.778" layer="27" display="off"/>
-<attribute name="MFGP" value="WS2812" x="21" y="0" size="1.778" layer="27" display="off"/>
-<attribute name="NOTES" value="DNP" x="21" y="0" size="1.778" layer="27" display="off"/>
+<attribute name="MFGP" value="WS2812S" x="21" y="0" size="1.778" layer="27" display="off"/>
+<attribute name="NOTES" value="" x="21" y="0" size="1.778" layer="27" display="off"/>
 </element>
 <element name="U$1" library="adafruit" package="FIDUCIAL_1MM" value="FIDUCIAL" x="-26.1" y="-10.4">
@@
 <via x="-18.3" y="-1.5" extent="1-16" drill="0.5"/>
 </signal>
-<signal name="+3V3" class="1">
+<signal name="+5V" class="1">
 <contactref element="U3" pad="8"/>
 <contactref element="U1" pad="3"/>
