File: POSCON.PCB Design Files/POSCON.PCB.sch (EAGLE design)
At the start: 27 parts, among them J1-PROG RJ45-8, J2 RJ45-8, U1 MC9S08QG-DT, U3 RS485SOIC, U4 PCA9552

Commit message: Finished power trace
Changed label to v1.1, fixed traces and moved vias / traces to
accomodate
Other:
- note added: "POSCON.PCB.v1.1"
- note removed: "POSCON.PCB.v1.0"
Changed lines of the file:
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@@
 <layer number="97" name="Info" color="7" fill="1" visible="yes" active="yes"/>
 <layer number="98" name="Guide" color="6" fill="1" visible="yes" active="yes"/>
+<layer number="99" name="SpiceOrder" color="5" fill="1" visible="yes" active="yes"/>
 <layer number="100" name="Muster" color="7" fill="1" visible="no" active="no"/>
 <layer number="101" name="Patch_Top" color="12" fill="4" visible="yes" active="yes"/>
@@
 <sheet>
 <plain>
-<text x="-218.44" y="-73.66" size="6.4516" layer="91">POSCON.PCB.v1.0</text>
+<text x="-218.44" y="-73.66" size="6.4516" layer="91">POSCON.PCB.v1.1</text>
 </plain>
 <instances>

Commit message: Prepare for release 1.2
Labelling, part names and numbers, new Gerbers and production documents
Parts:
- R.D2A, R.D2B, R.D2C, R.D2D: MFGP YC164-JR-07120RL -> YC164-JR-07620RL
- U1: value MC9S08QG-DT -> MC9S08SH8CTG; device GW-devices:MC9S08QG-DT -> GW-devices:MC9S08SH8CTG; MFGP MC9S08QG8CDTER -> MC9S08SH8CTG; PRICE 1.73 -> 2.00
Connections:
- net N$42: now also U1.PTA2; no longer U1.PTA2/KBIP2
- net N$43: now also U1.PTA1; no longer U1.PTA1/KBIP1
- net N$45: now also U1.PTA0; no longer U1.PTA0/KBIP0
Other:
- note added: "POSCON.PCB.v1.2"
- note removed: "POSCON.PCB.v1.1"
Changed lines of the file:
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@@
 </classes>
 <parts>
-<part name="U1" library="GW-devices" deviceset="MC9S08QG" device="-DT">
+<part name="U1" library="GW-devices" deviceset="MC9S08SH8CTG" device="">
 <attribute name="MFGN" value="Freescale"/>
-<attribute name="MFGP" value="MC9S08QG8CDTER"/>
-<attribute name="PRICE" value="1.73"/>
+<attribute name="MFGP" value="MC9S08SH8CTG"/>
+<attribute name="PRICE" value="2.00"/>
 </part>
 <part name="C1" library="GW-devices" deviceset="RF-C" device="0402" value=".1uF">
@@
 <part name="R.D2D" library="GW-devices" deviceset="RESISTOR-ARRAY-4X" device="-3216">
 <attribute name="MFGN" value="Yageo"/>
-<attribute name="MFGP" value="YC164-JR-07120RL"/>
+<attribute name="MFGP" value="YC164-JR-07620RL"/>
 <attribute name="PRICE" value="0.006"/>
 </part>
 <part name="R.D2C" library="GW-devices" deviceset="RESISTOR-ARRAY-4X" device="-3216">
 <attribute name="MFGN" value="Yageo"/>
-<attribute name="MFGP" value="YC164-JR-07120RL"/>
+<attribute name="MFGP" value="YC164-JR-07620RL"/>
 <attribute name="PRICE" value="0.006"/>
 </part>
 <part name="R.D2A" library="GW-devices" deviceset="RESISTOR-ARRAY-4X" device="-3216">
 <attribute name="MFGN" value="Yageo"/>
-<attribute name="MFGP" value="YC164-JR-07120RL"/>
+<attribute name="MFGP" value="YC164-JR-07620RL"/>
 <attribute name="PRICE" value="0.006"/>
 </part>
 <part name="R.D2B" library="GW-devices" deviceset="RESISTOR-ARRAY-4X" device="-3216">
 <attribute name="MFGN" value="Yageo"/>
-<attribute name="MFGP" value="YC164-JR-07120RL"/>
+<attribute name="MFGP" value="YC164-JR-07620RL"/>
 <attribute name="PRICE" value="0.006"/>
 </part>
@@
 <sheet>
 <plain>
-<text x="-218.44" y="-73.66" size="6.4516" layer="91">POSCON.PCB.v1.1</text>
+<text x="-218.44" y="-73.66" size="6.4516" layer="91">POSCON.PCB.v1.2</text>
 </plain>
 <instances>
@@
 <wire x1="116.84" y1="27.94" x2="58.42" y2="27.94" width="0.1524" layer="91"/>
 <wire x1="58.42" y1="27.94" x2="58.42" y2="25.4" width="0.1524" layer="91"/>
-<pinref part="U1" gate="G$1" pin="PTA2/KBIP2"/>
+<pinref part="U1" gate="G$1" pin="PTA2"/>
 <wire x1="58.42" y1="25.4" x2="58.42" y2="7.62" width="0.1524" layer="91"/>
 <wire x1="58.42" y1="7.62" x2="25.4" y2="7.62" width="0.1524" layer="91"/>
@@
 <wire x1="116.84" y1="43.18" x2="45.72" y2="43.18" width="0.1524" layer="91"/>
 <wire x1="45.72" y1="43.18" x2="45.72" y2="27.94" width="0.1524" layer="91"/>
-<pinref part="U1" gate="G$1" pin="PTA1/KBIP1"/>
+<pinref part="U1" gate="G$1" pin="PTA1"/>
 <wire x1="45.72" y1="27.94" x2="45.72" y2="12.7" width="0.1524" layer="91"/>
 <wire x1="45.72" y1="12.7" x2="25.4" y2="12.7" width="0.1524" layer="91"/>
@@
 <wire x1="116.84" y1="55.88" x2="25.4" y2="55.88" width="0.1524" layer="91"/>
 <junction x="116.84" y="55.88"/>
-<pinref part="U1" gate="G$1" pin="PTA0/KBIP0"/>
+<pinref part="U1" gate="G$1" pin="PTA0"/>
 <wire x1="25.4" y1="55.88" x2="25.4" y2="30.48" width="0.1524" layer="91"/>
 <pinref part="U$3" gate="G$1" pin="1"/>

Commit message: Fixing DRC
Residual Eagle errors on checklist
Connections:
- net N$19 renamed DIR
- net N$23 renamed RST
- net N$3 renamed LED_DI
- net N$42 renamed ACK
- net N$43 renamed INC_UP
- net N$45 renamed INC_DOWN
- net N$9 renamed BDM
- net SLA renamed SDA
- net SLC renamed SCL
Changed lines of the file:
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@@
 </segment>
 </net>
-<net name="N$19" class="0">
+<net name="DIR" class="0">
 <segment>
 <wire x1="50.8" y1="-35.56" x2="58.42" y2="-35.56" width="0.1524" layer="91"/>
@@
 </segment>
 </net>
-<net name="N$9" class="0">
+<net name="BDM" class="0">
 <segment>
 <wire x1="-55.88" y1="33.02" x2="-50.8" y2="33.02" width="0.1524" layer="91"/>
@@
 </segment>
 </net>
-<net name="N$23" class="0">
+<net name="RST" class="0">
 <segment>
 <wire x1="-71.12" y1="30.48" x2="-73.66" y2="30.48" width="0.1524" layer="91"/>
@@
 </segment>
 </net>
-<net name="SLC" class="0">
+<net name="SCL" class="0">
 <segment>
 <pinref part="U4" gate="G$1" pin="SCL"/>
@@
 </segment>
 </net>
-<net name="SLA" class="0">
+<net name="SDA" class="0">
 <segment>
 <pinref part="U4" gate="G$1" pin="SDA"/>
@@
 </segment>
 </net>
-<net name="N$42" class="0">
+<net name="ACK" class="0">
 <segment>
 <wire x1="116.84" y1="27.94" x2="119.38" y2="27.94" width="0.1524" layer="91"/>
@@
 </segment>
 </net>
-<net name="N$43" class="0">
+<net name="INC_UP" class="0">
 <segment>
 <wire x1="116.84" y1="43.18" x2="119.38" y2="43.18" width="0.1524" layer="91"/>
@@
 </segment>
 </net>
-<net name="N$45" class="0">
+<net name="INC_DOWN" class="0">
 <segment>
 <wire x1="116.84" y1="58.42" x2="119.38" y2="58.42" width="0.1524" layer="91"/>
@@
 </segment>
 </net>
-<net name="N$3" class="0">
+<net name="LED_DI" class="0">
 <segment>
 <pinref part="U$5" gate="G$1" pin="DI"/>

Commit message: Release v1.3
Fixed silkscreen (pin 1 markers), added WS2812S, added date / name to
fab text and updated all files correspondingly (BOM, ECO)
Parts:
- U$5: MFGP WS2812 -> WS2812S; NOTES DNP -> (none)
Connections:
- net +3V3 renamed +5V
Other:
- note added: "POSCON.PCB.v1.3"
- note removed: "POSCON.PCB.v1.2"
Changed lines of the file:
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@@
 </part>
 <part name="GND1" library="supply1" deviceset="GND" device=""/>
-<part name="+3V1" library="supply1" deviceset="+3V3" device=""/>
-<part name="+3V8" library="supply1" deviceset="+3V3" device=""/>
+<part name="+3V1" library="supply1" deviceset="+5V" device=""/>
+<part name="+3V8" library="supply1" deviceset="+5V" device=""/>
 <part name="GND8" library="supply1" deviceset="GND" device=""/>
 <part name="BDM" library="GW-devices" deviceset="TP2X4SMD" device="">
@@
 </part>
 <part name="GND4" library="supply1" deviceset="GND" device=""/>
-<part name="+3V4" library="supply1" deviceset="+3V3" device=""/>
+<part name="+3V4" library="supply1" deviceset="+5V" device=""/>
 <part name="U3" library="SparkFun" deviceset="RS485" device="SOIC">
 <attribute name="MFGN" value="TI"/>
@@
 <attribute name="PRICE" value="0.006"/>
 </part>
-<part name="+3V2" library="supply1" deviceset="+3V3" device=""/>
+<part name="+3V2" library="supply1" deviceset="+5V" device=""/>
 <part name="GND3" library="supply1" deviceset="GND" device=""/>
 <part name="R5" library="GW-devices" deviceset="RF-R" device="0402" value="10K">
@@
 <attribute name="PRICE" value="0.02"/>
 </part>
-<part name="+3V5" library="supply1" deviceset="+3V3" device=""/>
+<part name="+3V5" library="supply1" deviceset="+5V" device=""/>
 <part name="LED2" library="GW-devices" deviceset="7SEGMENT-1DIGIT" device="SMD">
 <attribute name="MFGN" value="Kingbright"/>
@@
 <attribute name="MFGP" value="ACSA04-41SEKWA-F01 "/>
 </part>
-<part name="+3V3" library="supply1" deviceset="+3V3" device=""/>
-<part name="+3V6" library="supply1" deviceset="+3V3" device=""/>
+<part name="+3V3" library="supply1" deviceset="+5V" device=""/>
+<part name="+3V6" library="supply1" deviceset="+5V" device=""/>
 <part name="GND5" library="supply1" deviceset="GND" device=""/>
 <part name="SW-ACK" library="GW-devices" deviceset="SWITCH-TACTILE" device="-320.01E11WHT">
@@
 <part name="U$5" library="GW-devices" deviceset="WS2812" device="">
 <attribute name="MFGN" value="Worldsemi"/>
-<attribute name="MFGP" value="WS2812"/>
-<attribute name="NOTES" value="DNP"/>
+<attribute name="MFGP" value="WS2812S"/>
+<attribute name="NOTES" value=""/>
 </part>
 <part name="GND2" library="supply1" deviceset="GND" device=""/>
-<part name="+3V7" library="supply1" deviceset="+3V3" device=""/>
+<part name="+3V7" library="supply1" deviceset="+5V" device=""/>
 <part name="U$1" library="adafruit" deviceset="FIDUCIAL" device="">
 <attribute name="NOTES" value="DNP"/>
@@
 <sheet>
 <plain>
-<text x="-218.44" y="-73.66" size="6.4516" layer="91">POSCON.PCB.v1.2</text>
+<text x="-218.44" y="-73.66" size="6.4516" layer="91">POSCON.PCB.v1.3</text>
 </plain>
 <instances>
@@
 </instance>
 <instance part="GND1" gate="1" x="-33.02" y="-45.72"/>
-<instance part="+3V1" gate="G$1" x="-33.02" y="45.72"/>
-<instance part="+3V8" gate="G$1" x="91.44" y="-17.78"/>
+<instance part="+3V1" gate="1" x="-33.02" y="45.72"/>
+<instance part="+3V8" gate="1" x="91.44" y="-17.78"/>
 <instance part="GND8" gate="1" x="91.44" y="-50.8"/>
 <instance part="BDM" gate="G$1" x="-63.5" y="30.48" smashed="yes" rot="MR0">
@@
 </instance>
 <instance part="GND4" gate="1" x="-86.36" y="53.34" rot="R180"/>
-<instance part="+3V4" gate="G$1" x="-86.36" y="10.16" rot="R180"/>
+<instance part="+3V4" gate="1" x="-86.36" y="10.16" rot="R180"/>
 <instance part="U3" gate="G$1" x="68.58" y="-33.02">
 <attribute name="MFGN" x="68.58" y="-33.02" size="1.778" layer="96" display="off"/>
@@
 <attribute name="PRICE" x="-246.38" y="121.92" size="1.778" layer="96" rot="R90" display="off"/>
 </instance>
-<instance part="+3V2" gate="G$1" x="-73.66" y="-2.54"/>
+<instance part="+3V2" gate="1" x="-73.66" y="-2.54"/>
 <instance part="GND3" gate="1" x="-106.68" y="116.84" rot="R180"/>
 <instance part="R5" gate="G$1" x="-83.82" y="-20.32">
@@
 <attribute name="PRICE" x="-83.82" y="-10.16" size="1.778" layer="96" display="off"/>
 </instance>
-<instance part="+3V5" gate="G$1" x="-73.66" y="81.28"/>
+<instance part="+3V5" gate="1" x="-73.66" y="81.28"/>
 <instance part="LED2" gate="G$1" x="-274.32" y="81.28">
 <attribute name="MFGN" x="-274.32" y="81.28" size="1.778" layer="96" display="off"/>
@@
 <attribute name="MFGP" x="-243.84" y="81.28" size="1.778" layer="96" display="off"/>
 </instance>
-<instance part="+3V3" gate="G$1" x="-307.34" y="109.22"/>
-<instance part="+3V6" gate="G$1" x="-307.34" y="60.96"/>
+<instance part="+3V3" gate="1" x="-307.34" y="109.22"/>
+<instance part="+3V6" gate="1" x="-307.34" y="60.96"/>
 <instance part="GND5" gate="1" x="144.78" y="7.62"/>
 <instance part="SW-ACK" gate="G$1" x="124.46" y="27.94"/>
@@
 </instance>
 <instance part="GND2" gate="1" x="-7.62" y="-81.28"/>
-<instance part="+3V7" gate="G$1" x="7.62" y="-43.18"/>
+<instance part="+3V7" gate="1" x="7.62" y="-43.18"/>
 <instance part="U$1" gate="G$1" x="-33.02" y="134.62">
 <attribute name="NOTES" x="-33.02" y="134.62" size="1.778" layer="96" display="off"/>
@@
 </segment>
 </net>
-<net name="+3V3" class="1">
+<net name="+5V" class="1">
 <segment>
 <wire x1="83.82" y1="-30.48" x2="91.44" y2="-30.48" width="0.1524" layer="91"/>
 <wire x1="91.44" y1="-30.48" x2="91.44" y2="-20.32" width="0.1524" layer="91"/>
 <junction x="91.44" y="-30.48"/>
-<pinref part="+3V8" gate="G$1" pin="+3V3"/>
+<pinref part="+3V8" gate="1" pin="+5V"/>
 <pinref part="U3" gate="G$1" pin="VCC"/>
 <wire x1="157.48" y1="-10.16" x2="139.7" y2="-10.16" width="0.1524" layer="91"/>
@@
 <pinref part="U1" gate="G$1" pin="VDD"/>
 <pinref part="C1" gate="G$1" pin="1"/>
-<pinref part="+3V1" gate="G$1" pin="+3V3"/>
+<pinref part="+3V1" gate="1" pin="+5V"/>
 <pinref part="R1" gate="G$1" pin="2"/>
 </segment>
@@
 <wire x1="-86.36" y1="27.94" x2="-86.36" y2="12.7" width="0.1524" layer="91"/>
 <pinref part="BDM" gate="G$1" pin="6"/>
-<pinref part="+3V4" gate="G$1" pin="+3V3"/>
+<pinref part="+3V4" gate="1" pin="+5V"/>
 </segment>
 <segment>
@@
 <wire x1="-73.66" y1="-20.32" x2="-73.66" y2="-10.16" width="0.1524" layer="91"/>
 <junction x="-73.66" y="-10.16"/>
-<pinref part="+3V2" gate="G$1" pin="+3V3"/>
+<pinref part="+3V2" gate="1" pin="+5V"/>
 <pinref part="R6" gate="G$1" pin="2"/>
 <pinref part="R5" gate="G$1" pin="2"/>
@@
 <wire x1="-73.66" y1="66.04" x2="-73.66" y2="78.74" width="0.1524" layer="91"/>
 <pinref part="U4" gate="G$1" pin="VCC"/>
-<pinref part="+3V5" gate="G$1" pin="+3V3"/>
+<pinref part="+3V5" gate="1" pin="+5V"/>
 </segment>
 <segment>
@@
 <wire x1="-276.86" y1="55.88" x2="-307.34" y2="55.88" width="0.1524" layer="91"/>
 <junction x="-276.86" y="55.88"/>
-<pinref part="+3V6" gate="G$1" pin="+3V3"/>
+<pinref part="+3V6" gate="1" pin="+5V"/>
 <wire x1="-307.34" y1="55.88" x2="-307.34" y2="58.42" width="0.1524" layer="91"/>
 </segment>
@@
 <wire x1="-276.86" y1="104.14" x2="-307.34" y2="104.14" width="0.1524" layer="91"/>
 <junction x="-276.86" y="104.14"/>
-<pinref part="+3V3" gate="G$1" pin="+3V3"/>
+<pinref part="+3V3" gate="1" pin="+5V"/>
 <wire x1="-307.34" y1="104.14" x2="-307.34" y2="106.68" width="0.1524" layer="91"/>
 </segment>
@@
 <pinref part="U$5" gate="G$1" pin="VCC"/>
 <wire x1="25.4" y1="-60.96" x2="22.86" y2="-60.96" width="0.1524" layer="91"/>
-<pinref part="+3V7" gate="G$1" pin="+3V3"/>
+<pinref part="+3V7" gate="1" pin="+5V"/>
 <wire x1="7.62" y1="-45.72" x2="7.62" y2="-48.26" width="0.1524" layer="91"/>
 <junction x="7.62" y="-48.26"/>
