File: INKY.PCB Design Files/INKY.PCB.sch (EAGLE design)
At the start: 34 parts, among them J1-PROG RJ45-8, J2 RJ45-8, U1 MC9S08SH8CTG, U3 RS485SOIC

Commit message: Still routing
~ 95% done
Changed lines of the file:
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@@
-<attribute name="NOTES" value="DNP"/>
-</part>
-<part name="U$2" library="adafruit" deviceset="FIDUCIAL" device="">
 <attribute name="NOTES" value="DNP"/>
 </part>
@@
 </part>
 <part name="U$7" library="adafruit" deviceset="FIDUCIAL" device="">
-<attribute name="NOTES" value="DNP"/>
-</part>
-<part name="U$8" library="adafruit" deviceset="FIDUCIAL" device="">
 <attribute name="NOTES" value="DNP"/>
 </part>
@@
 <attribute name="MFGP" value="CRCW080510K0FKEB"/>
 </part>
+<part name="U$2" library="adafruit" deviceset="FIDUCIAL" device="">
+<attribute name="NOTES" value="DNP"/>
+</part>
+<part name="U$8" library="adafruit" deviceset="FIDUCIAL" device="">
+<attribute name="NOTES" value="DNP"/>
+</part>
 </parts>
 <sheets>
@@
 <attribute name="NOTES" x="-33.02" y="134.62" size="1.778" layer="96" display="off"/>
 </instance>
-<instance part="U$2" gate="G$1" x="0" y="134.62">
-<attribute name="NOTES" x="0" y="134.62" size="1.778" layer="96" display="off"/>
-</instance>
 <instance part="U$6" gate="G$1" x="30.48" y="132.08">
 <attribute name="NOTES" x="30.48" y="132.08" size="1.778" layer="96" display="off"/>
@@
 <instance part="U$7" gate="G$1" x="-25.4" y="109.22">
 <attribute name="NOTES" x="-25.4" y="109.22" size="1.778" layer="96" display="off"/>
-</instance>
-<instance part="U$8" gate="G$1" x="5.08" y="104.14">
-<attribute name="NOTES" x="5.08" y="104.14" size="1.778" layer="96" display="off"/>
 </instance>
 <instance part="U$9" gate="G$1" x="33.02" y="104.14">
@@
 <attribute name="MFGP" x="2.54" y="-104.14" size="1.778" layer="96" display="off"/>
 </instance>
+<instance part="U$2" gate="G$1" x="-25.4" y="91.44">
+<attribute name="NOTES" x="-25.4" y="91.44" size="1.778" layer="96" display="off"/>
+</instance>
+<instance part="U$8" gate="G$1" x="33.02" y="88.9">
+<attribute name="NOTES" x="33.02" y="88.9" size="1.778" layer="96" display="off"/>
+</instance>
 </instances>

Commit message: Inky finishing
Done routing, need to fix angles.
Parts:
- J1-PROG, J2: value RJ45-8 -> RJ45-8MOLEX_0955406886; device GW-devices:RJ45-8 -> GW-devices:RJ45-8MOLEX_0955406886; MFGN Molex -> (none); MFGP 0955016889 -> (none)
- SW-ACK: value SWITCH-TACTILE-320.01E11WHT -> SWITCH-TACTILE-5E/5GSH9; device GW-devices:SWITCH-TACTILE-320.01E11WHT -> GW-devices:SWITCH-TACTILE-5E/5GSH9; MFGP 320.01E11WHT -> (none)
- U$10: value 52745-1097 -> (none)
Connections:
- removed net +3V3: U$10.P$5, U$10.P$6, U$10.P$7, U$12.1, U$13.VOUT, U$14.OE, U$14.VCCA, U$15.2, U$17.1, U$18.1, U$24.1
- new net GMD: U$10.DISP, U$10.VDD, U$10.VDDA, U$12.1, U$13.VOUT, U$14.OE, U$14.VCCA, U$15.2, U$17.1, U$18.1, U$24.1
- net ACK: no longer SW-ACK.2
- net GND: now also U$10.VSS, U$10.VSSA; no longer U$10.P$10, U$10.P$9
- net N$2: now also U$10.SCLK; no longer U$10.P$1
- net N$3: now also U$10.SI; no longer U$10.P$2
- net N$32: now also U$10.EXTMODE; no longer U$10.P$8
- net N$33: now also U$10.EXCOMIN; no longer U$10.P$4
- net N$4: now also U$10.SCS; no longer U$10.P$3
Changed lines of the file:
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@@
 </part>
 <part name="GND5" library="supply1" deviceset="GND" device=""/>
-<part name="SW-ACK" library="GW-devices" deviceset="SWITCH-TACTILE" device="-320.01E11WHT">
-<attribute name="MFGP" value="320.01E11WHT"/>
-</part>
+<part name="SW-ACK" library="GW-devices" deviceset="SWITCH-TACTILE" device="-5E/5GSH9" value="SWITCH-TACTILE-5E/5GSH9"/>
 <part name="U$3" library="GW-devices" deviceset="SWITCH-TACTILE" device="" value="SWITCH-TACTILE">
 <attribute name="MFGN" value="E-Switch"/>
@@
 <attribute name="MFGP" value="TL3301PF160QG"/>
 </part>
-<part name="J1-PROG" library="GW-devices" deviceset="RJ45-8" device="">
-<attribute name="MFGN" value="Molex"/>
-<attribute name="MFGP" value="0955016889"/>
+<part name="J1-PROG" library="GW-devices" deviceset="RJ45-8" device="MOLEX_0955406886" value="RJ45-8MOLEX_0955406886">
 <attribute name="PRICE" value="0.89"/>
 </part>
-<part name="J2" library="GW-devices" deviceset="RJ45-8" device="">
-<attribute name="MFGN" value="Molex"/>
-<attribute name="MFGP" value="0955016889"/>
+<part name="J2" library="GW-devices" deviceset="RJ45-8" device="MOLEX_0955406886" value="RJ45-8MOLEX_0955406886">
 <attribute name="PRICE" value="0.89"/>
 </part>
@@
 <attribute name="NOTES" value="DNP"/>
 </part>
-<part name="U$6" library="adafruit" deviceset="FIDUCIAL" device="">
-<attribute name="NOTES" value="DNP"/>
-</part>
 <part name="U$7" library="adafruit" deviceset="FIDUCIAL" device="">
-<attribute name="NOTES" value="DNP"/>
-</part>
-<part name="U$9" library="adafruit" deviceset="FIDUCIAL" device="">
 <attribute name="NOTES" value="DNP"/>
 </part>
@@
 <attribute name="NOTES" value="DNP"/>
 </part>
+<part name="U$6" library="adafruit" deviceset="FIDUCIAL" device="">
+<attribute name="NOTES" value="DNP"/>
+</part>
+<part name="U$9" library="adafruit" deviceset="FIDUCIAL" device="">
+<attribute name="NOTES" value="DNP"/>
+</part>
 </parts>
 <sheets>
@@
 </instance>
 <instance part="J1-PROG" gate="G$1" x="170.18" y="-20.32">
-<attribute name="MFGN" x="170.18" y="-20.32" size="1.778" layer="96" display="off"/>
-<attribute name="MFGP" x="170.18" y="-20.32" size="1.778" layer="96" display="off"/>
 <attribute name="PRICE" x="170.18" y="-20.32" size="1.778" layer="96" display="off"/>
 </instance>
 <instance part="J2" gate="G$1" x="170.18" y="-66.04">
-<attribute name="MFGN" x="170.18" y="-66.04" size="1.778" layer="96" display="off"/>
-<attribute name="MFGP" x="170.18" y="-66.04" size="1.778" layer="96" display="off"/>
 <attribute name="PRICE" x="170.18" y="-66.04" size="1.778" layer="96" display="off"/>
 </instance>
@@
 <attribute name="NOTES" x="-33.02" y="134.62" size="1.778" layer="96" display="off"/>
 </instance>
-<instance part="U$6" gate="G$1" x="30.48" y="132.08">
-<attribute name="NOTES" x="30.48" y="132.08" size="1.778" layer="96" display="off"/>
-</instance>
 <instance part="U$7" gate="G$1" x="-25.4" y="109.22">
 <attribute name="NOTES" x="-25.4" y="109.22" size="1.778" layer="96" display="off"/>
-</instance>
-<instance part="U$9" gate="G$1" x="33.02" y="104.14">
-<attribute name="NOTES" x="33.02" y="104.14" size="1.778" layer="96" display="off"/>
 </instance>
 <instance part="U$10" gate="G$1" x="-213.36" y="-22.86" rot="R270">
@@
 <instance part="U$8" gate="G$1" x="33.02" y="88.9">
 <attribute name="NOTES" x="33.02" y="88.9" size="1.778" layer="96" display="off"/>
+</instance>
+<instance part="U$6" gate="G$1" x="-7.62" y="134.62">
+<attribute name="NOTES" x="-7.62" y="134.62" size="1.778" layer="96" display="off"/>
+</instance>
+<instance part="U$9" gate="G$1" x="-2.54" y="111.76">
+<attribute name="NOTES" x="-2.54" y="111.76" size="1.778" layer="96" display="off"/>
 </instance>
 </instances>
@@
 <wire x1="132.08" y1="43.18" x2="132.08" y2="40.64" width="0.1524" layer="91"/>
 <wire x1="132.08" y1="40.64" x2="129.54" y2="40.64" width="0.1524" layer="91"/>
-<wire x1="132.08" y1="27.94" x2="132.08" y2="25.4" width="0.1524" layer="91"/>
-<wire x1="132.08" y1="25.4" x2="129.54" y2="25.4" width="0.1524" layer="91"/>
 <wire x1="132.08" y1="58.42" x2="132.08" y2="55.88" width="0.1524" layer="91"/>
 <wire x1="132.08" y1="55.88" x2="129.54" y2="55.88" width="0.1524" layer="91"/>
@@
 <junction x="132.08" y="58.42"/>
 <pinref part="GND5" gate="1" pin="GND"/>
-<pinref part="SW-ACK" gate="G$1" pin="4"/>
 <pinref part="SW-ACK" gate="G$1" pin="3"/>
 <pinref part="U$3" gate="G$1" pin="3"/>
@@
 <pinref part="U$4" gate="G$1" pin="3"/>
 <pinref part="U$4" gate="G$1" pin="4"/>
-</segment>
-<segment>
-<pinref part="U$10" gate="G$1" pin="P$10"/>
+<pinref part="SW-ACK" gate="G$1" pin="4"/>
+<wire x1="129.54" y1="25.4" x2="132.08" y2="25.4" width="0.1524" layer="91"/>
+<wire x1="132.08" y1="25.4" x2="132.08" y2="27.94" width="0.1524" layer="91"/>
+</segment>
+<segment>
+<pinref part="U$10" gate="G$1" pin="VSSA"/>
 <wire x1="-208.28" y1="-33.02" x2="-203.2" y2="-33.02" width="0.1524" layer="91"/>
 <wire x1="-203.2" y1="-33.02" x2="-203.2" y2="-30.48" width="0.1524" layer="91"/>
-<pinref part="U$10" gate="G$1" pin="P$9"/>
+<pinref part="U$10" gate="G$1" pin="VSS"/>
 <wire x1="-203.2" y1="-30.48" x2="-208.28" y2="-30.48" width="0.1524" layer="91"/>
 <wire x1="-203.2" y1="-33.02" x2="-203.2" y2="-38.1" width="0.1524" layer="91"/>
@@
 <net name="ACK" class="0">
 <segment>
-<wire x1="116.84" y1="27.94" x2="119.38" y2="27.94" width="0.1524" layer="91"/>
-<wire x1="116.84" y1="27.94" x2="116.84" y2="25.4" width="0.1524" layer="91"/>
-<wire x1="116.84" y1="25.4" x2="119.38" y2="25.4" width="0.1524" layer="91"/>
-<junction x="116.84" y="27.94"/>
 <pinref part="SW-ACK" gate="G$1" pin="1"/>
-<pinref part="SW-ACK" gate="G$1" pin="2"/>
-<wire x1="116.84" y1="27.94" x2="58.42" y2="27.94" width="0.1524" layer="91"/>
+<wire x1="119.38" y1="27.94" x2="58.42" y2="27.94" width="0.1524" layer="91"/>
 <wire x1="58.42" y1="27.94" x2="58.42" y2="25.4" width="0.1524" layer="91"/>
 <pinref part="U1" gate="G$1" pin="PTA2"/>
@@
 <net name="N$32" class="0">
 <segment>
-<pinref part="U$10" gate="G$1" pin="P$8"/>
+<pinref part="U$10" gate="G$1" pin="EXTMODE"/>
 <pinref part="U$11" gate="G$1" pin="1"/>
 <wire x1="-208.28" y1="-27.94" x2="-195.58" y2="-27.94" width="0.1524" layer="91"/>
@@
 <net name="N$33" class="0">
 <segment>
-<pinref part="U$10" gate="G$1" pin="P$4"/>
+<pinref part="U$10" gate="G$1" pin="EXCOMIN"/>
 <pinref part="U$25" gate="G$1" pin="1"/>
 <wire x1="-208.28" y1="-17.78" x2="-160.02" y2="-17.78" width="0.1524" layer="91"/>
@@
 </segment>
 </net>
-<net name="+3V3" class="3">
-<segment>
-<pinref part="U$10" gate="G$1" pin="P$5"/>
+<net name="GMD" class="3">
+<segment>
+<pinref part="U$10" gate="G$1" pin="DISP"/>
 <wire x1="-208.28" y1="-20.32" x2="-193.04" y2="-20.32" width="0.1524" layer="91"/>
 <wire x1="-193.04" y1="-20.32" x2="-187.96" y2="-20.32" width="0.1524" layer="91"/>
@@
 <wire x1="-167.64" y1="-22.86" x2="-162.56" y2="-22.86" width="0.1524" layer="91"/>
 <pinref part="U$12" gate="G$1" pin="1"/>
-<pinref part="U$10" gate="G$1" pin="P$7"/>
+<pinref part="U$10" gate="G$1" pin="VDD"/>
 <wire x1="-208.28" y1="-25.4" x2="-195.58" y2="-25.4" width="0.1524" layer="91"/>
 <wire x1="-195.58" y1="-25.4" x2="-193.04" y2="-25.4" width="0.1524" layer="91"/>
 <wire x1="-193.04" y1="-25.4" x2="-193.04" y2="-22.86" width="0.1524" layer="91"/>
-<pinref part="U$10" gate="G$1" pin="P$6"/>
+<pinref part="U$10" gate="G$1" pin="VDDA"/>
 <wire x1="-193.04" y1="-22.86" x2="-208.28" y2="-22.86" width="0.1524" layer="91"/>
 <wire x1="-193.04" y1="-22.86" x2="-193.04" y2="-20.32" width="0.1524" layer="91"/>
@@
 <net name="N$2" class="0">
 <segment>
-<pinref part="U$10" gate="G$1" pin="P$1"/>
+<pinref part="U$10" gate="G$1" pin="SCLK"/>
 <wire x1="-170.18" y1="-10.16" x2="-208.28" y2="-10.16" width="0.1524" layer="91"/>
 <wire x1="-170.18" y1="-10.16" x2="-165.1" y2="-10.16" width="0.1524" layer="91"/>
@@
 <net name="N$3" class="0">
 <segment>
-<pinref part="U$10" gate="G$1" pin="P$2"/>
+<pinref part="U$10" gate="G$1" pin="SI"/>
 <wire x1="-167.64" y1="-12.7" x2="-208.28" y2="-12.7" width="0.1524" layer="91"/>
 <pinref part="U$14" gate="G$1" pin="P$3"/>
@@
 <net name="N$4" class="0">
 <segment>
-<pinref part="U$10" gate="G$1" pin="P$3"/>
+<pinref part="U$10" gate="G$1" pin="SCS"/>
 <wire x1="-162.56" y1="-15.24" x2="-208.28" y2="-15.24" width="0.1524" layer="91"/>
 <wire x1="-162.56" y1="-15.24" x2="-144.78" y2="-15.24" width="0.1524" layer="91"/>

Commit message: Inky v0.1
Parts:
- U3: MFGN TI -> (none)
Changed lines of the file:
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@@
 <part name="+3V4" library="supply1" deviceset="+5V" device=""/>
 <part name="U3" library="SparkFun" deviceset="RS485" device="SOIC">
-<attribute name="MFGN" value="TI"/>
 <attribute name="MFGP" value="SN65HVD1781DR"/>
 <attribute name="PRICE" value="4.29"/>

Commit message: Inky 0.2
Parts:
- U$11, U$25: value (none) -> 10K
Connections:
- net INC_DOWN: no longer U$3.2
Other:
- note added: "INKY.PCB.v1.0P2"
- note removed: "INKY.PCB.v1.0P1"
Changed lines of the file:
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@@
 <attribute name="MFGP" value="52745-1097"/>
 </part>
-<part name="U$11" library="GW-devices" deviceset="RF-R" device="0805">
+<part name="U$11" library="GW-devices" deviceset="RF-R" device="0805" value="10K">
 <attribute name="MFGP" value="CRCW080510K0FKEB"/>
 </part>
@@
 <attribute name="MFGP" value="0805YD104KAT2A"/>
 </part>
-<part name="U$25" library="GW-devices" deviceset="RF-R" device="0805">
+<part name="U$25" library="GW-devices" deviceset="RF-R" device="0805" value="10K">
 <attribute name="MFGP" value="CRCW080510K0FKEB"/>
 </part>
@@
 <sheet>
 <plain>
-<text x="-218.44" y="-73.66" size="6.4516" layer="91">INKY.PCB.v1.0P1</text>
+<text x="-218.44" y="-73.66" size="6.4516" layer="91">INKY.PCB.v1.0P2</text>
 </plain>
 <instances>
@@
 <wire x1="116.84" y1="58.42" x2="119.38" y2="58.42" width="0.1524" layer="91"/>
 <wire x1="116.84" y1="58.42" x2="116.84" y2="55.88" width="0.1524" layer="91"/>
-<wire x1="116.84" y1="55.88" x2="119.38" y2="55.88" width="0.1524" layer="91"/>
 <wire x1="116.84" y1="55.88" x2="25.4" y2="55.88" width="0.1524" layer="91"/>
 <junction x="116.84" y="55.88"/>
@@
 <wire x1="25.4" y1="55.88" x2="25.4" y2="30.48" width="0.1524" layer="91"/>
 <pinref part="U$3" gate="G$1" pin="1"/>
-<pinref part="U$3" gate="G$1" pin="2"/>
 <wire x1="25.4" y1="30.48" x2="25.4" y2="17.78" width="0.1524" layer="91"/>
 <wire x1="25.4" y1="30.48" x2="-55.88" y2="30.48" width="0.1524" layer="91"/>
